File: tinyShield.sch (EAGLE design)
At the start: 12 parts, among them J1 TSW-103-07-L-SNO_SILK, J2 TSW-103-07-L-SNO_SILK, J3 TSW-103-07-L-SNO_SILK, U1 3M 214-3339-00

Commit message: Added SW1 to switch 5V power from host Arduino; Update hardware rev to B
Parts:
- added SW1: CL-SB-12B, C3-Switches:CL-SB-12B
Connections:
- new net VCC: C1.1, SW1.3, U$8ICSP.5V$1, U1.1, U1.11
- net +5V: now also SW1.2; no longer C1.1, U$8ICSP.5V$1, U1.1, U1.11
Other:
- moved on the sheet: C1
